File: antenna_top_cap_v2/antenna_top_cap_v2.kicad_sch (KiCad schematic)
At the start: 56 parts, among them IC1 PCT2075DP,118, J1 Battery Charge Bypass, J10 BM04B-SRSS-TB(LF)(SN), J12 BM04B-SRSS-TB(LF)(SN), J12 FC Board Connector, J14 BM04B-SRSS-TB(LF)(SN), J16 BM04B-SRSS-TB(LF)(SN), J19 EPS Board Connector, J2 EPS USB Bootselect Jumper, J20 FC USB Bootselect Jumper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

Commit message: Completed Layout
Connections:
- net BURN: now also J7.1 (Power); no longer J7.2 (GND)
- net GND: no longer J19.12 (Pin_12), J7.1 (Power)
- new net BURN_GND: J19.12 (Pin_12), J7.2 (GND)
Other:
- moved on the sheet: J7
Changed lines of the file:
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@@
 	(wire
 		(pts
-			(xy 125.73 21.59) (xy 121.92 21.59)
-		)
-		(stroke
-			(width 0)
-			(type default)
-		)
-	)
-	(wire
-		(pts
 			(xy 222.377 147.32) (xy 241.3 147.32)
 		)
@@
 	(wire
 		(pts
-			(xy 110.49 138.43) (xy 110.49 139.7)
-		)
-		(stroke
-			(width 0)
-			(type default)
-		)
-	)
-	(wire
-		(pts
 			(xy 205.74 36.83) (xy 205.74 45.72)
 		)
@@
 	(wire
 		(pts
-			(xy 121.92 21.59) (xy 121.92 26.67)
-		)
-		(stroke
-			(width 0)
-			(type default)
-		)
-	)
-	(wire
-		(pts
 			(xy 242.57 33.02) (xy 242.57 40.64)
 		)
@@
 	(wire
 		(pts
-			(xy 119.38 20.32) (xy 125.73 20.32)
-		)
-		(stroke
-			(width 0)
-			(type default)
-		)
-	)
-	(wire
-		(pts
 			(xy 39.37 85.09) (xy 52.324 85.09)
 		)
@@
 	(wire
 		(pts
-			(xy 106.68 138.43) (xy 110.49 138.43)
-		)
-		(stroke
-			(width 0)
-			(type default)
-		)
-	)
-	(wire
-		(pts
 			(xy 90.17 83.82) (xy 85.471 83.82)
 		)
@@
 	(wire
 		(pts
-			(xy 106.68 161.29) (xy 106.68 138.43)
+			(xy 116.84 21.59) (xy 130.81 21.59)
 		)
 		(stroke
@@
 	(wire
 		(pts
+			(xy 130.81 20.32) (xy 129.54 20.32)
+		)
+		(stroke
+			(width 0)
+			(type default)
+		)
+	)
+	(wire
+		(pts
 			(xy 29.21 50.8) (xy 29.21 55.118)
 		)
@@
 		)
 	)
+	(global_label "BURN_GND"
+		(shape output)
+		(at 106.68 161.29 90)
+		(fields_autoplaced yes)
+		(effects
+			(font
+				(size 1.27 1.27)
+			)
+			(justify left)
+		)
+		(property "Intersheetrefs" "${INTERSHEET_REFS}"
+			(at 106.68 148.2657 90)
+			(effects
+				(font
+					(size 1.27 1.27)
+				)
+				(justify left)
+				(hide yes)
+			)
+		)
+	)
 	(global_label "~{FC_RESET}"
 		(shape output)
@@
 		)
 	)
+	(global_label "BURN_GND"
+		(shape output)
+		(at 129.54 20.32 180)
+		(fields_autoplaced yes)
+		(effects
+			(font
+				(size 1.27 1.27)
+			)
+			(justify right)
+		)
+		(property "Intersheetrefs" "${INTERSHEET_REFS}"
+			(at 116.5157 20.32 0)
+			(effects
+				(font
+					(size 1.27 1.27)
+				)
+				(justify right)
+				(hide yes)
+			)
+		)
+	)
 	(global_label "EPS_USB_D-"
 		(shape input)
@@
 	(global_label "BURN"
 		(shape input)
-		(at 119.38 20.32 180)
+		(at 116.84 21.59 180)
 		(fields_autoplaced yes)
 		(effects
@@
 		)
 		(property "Intersheetrefs" "${INTERSHEET_REFS}"
-			(at 111.1938 20.32 0)
+			(at 108.6538 21.59 0)
 			(effects
 				(font
@@
 	)
 	(symbol
-		(lib_name "GND_3")
-		(lib_id "power:GND")
-		(at 121.92 26.67 0)
-		(unit 1)
-		(exclude_from_sim no)
-		(in_bom yes)
-		(on_board yes)
-		(dnp no)
-		(property "Reference" "#PWR023"
-			(at 121.92 33.02 0)
-			(effects
-				(font
-					(size 1.27 1.27)
-				)
-				(hide yes)
-			)
-		)
-		(property "Value" "GND"
-			(at 125.73 28.448 0)
-			(effects
-				(font
-					(size 1.27 1.27)
-				)
-			)
-		)
-		(property "Footprint" ""
-			(at 121.92 26.67 0)
-			(effects
-				(font
-					(size 1.27 1.27)
-				)
-				(hide yes)
-			)
-		)
-		(property "Datasheet" ""
-			(at 121.92 26.67 0)
-			(effects
-				(font
-					(size 1.27 1.27)
-				)
-				(hide yes)
-			)
-		)
-		(property "Description" "Power symbol creates a global label with name \"GND\" , ground"
-			(at 121.92 26.67 0)
-			(effects
-				(font
-					(size 1.27 1.27)
-				)
-				(hide yes)
-			)
-		)
-		(pin "1"
-		)
-		(instances
-			(project "antenna_top_cap_v2"
-				(path "/e63e39d7-6ac0-4ffd-8aa3-1841a4541b55"
-					(reference "#PWR023")
-					(unit 1)
-				)
-			)
-		)
-	)
-	(symbol
 		(lib_id "Adafruit VL6180 Time of Flight Sensor-eagle-import:CAP_CERAMIC0805-NOOUTLINE")
 		(at 238.76 33.02 0)
@@
 	)
 	(symbol
-		(lib_name "GND_1")
-		(lib_id "power:GND")
-		(at 110.49 139.7 0)
-		(unit 1)
-		(exclude_from_sim no)
-		(in_bom yes)
-		(on_board yes)
-		(dnp no)
-		(property "Reference" "#PWR021"
-			(at 110.49 146.05 0)
-			(effects
-				(font
-					(size 1.27 1.27)
-				)
-				(hide yes)
-			)
-		)
-		(property "Value" "GND"
-			(at 110.49 144.018 0)
-			(effects
-				(font
-					(size 1.27 1.27)
-				)
-			)
-		)
-		(property "Footprint" ""
-			(at 110.49 139.7 0)
-			(effects
-				(font
-					(size 1.27 1.27)
-				)
-				(hide yes)
-			)
-		)
-		(property "Datasheet" ""
-			(at 110.49 139.7 0)
-			(effects
-				(font
-					(size 1.27 1.27)
-				)
-				(hide yes)
-			)
-		)
-		(property "Description" "Power symbol creates a global label with name \"GND\" , ground"
-			(at 110.49 139.7 0)
-			(effects
-				(font
-					(size 1.27 1.27)
-				)
-				(hide yes)
-			)
-		)
-		(pin "1"
-		)
-		(instances
-			(project "antenna_top_cap_v2"
-				(path "/e63e39d7-6ac0-4ffd-8aa3-1841a4541b55"
-					(reference "#PWR021")
-					(unit 1)
-				)
-			)
-		)
-	)
-	(symbol
 		(lib_id "Adafruit ItsyBitsy RP2040-eagle-import:RESISTOR_0402NO")
 		(at 17.272 84.963 270)
@@
 	(symbol
 		(lib_id "Antenna:Burn_Wire")
-		(at 125.73 21.59 180)
+		(at 130.81 21.59 180)
 		(unit 1)
 		(exclude_from_sim no)
@@
 		(fields_autoplaced yes)
 		(property "Reference" "J7"
-			(at 128.788 23.368 0)
+			(at 133.868 23.368 0)
 			(effects
 				(font
@@
 		)
 		(property "Value" "~"
-			(at 119.888 19.177 0)
+			(at 124.968 19.177 0)
 			(effects
 				(font
@@
 		)
 		(property "Footprint" "Antenna_board:Burn_Wire"
-			(at 119.888 19.177 0)
+			(at 124.968 19.177 0)
 			(effects
 				(font
@@
 		)
 		(property "Datasheet" ""
-			(at 119.888 19.177 0)
+			(at 124.968 19.177 0)
 			(effects
 				(font
@@
 		)
 		(property "Description" ""
-			(at 125.73 21.59 0)
+			(at 130.81 21.59 0)
 			(effects
 				(font
