File: antenna_top_cap_v2b_cygnet_special/antenna_top_cap_v2b_cygnet_special.kicad_pcb (KiCad board)
At the start: 4 copper layers, 100 x 100 mm, 57 parts, among them J1 DEBUG, J10 WDT Disable Jumper, J11 DF11-4DP-2DSA, J12 USB_C_Receptacle_USB2.0_16P, J13 DNP, J2 Battery Charge Bypass, J3 FC Reset Jumper, J4 FC USB Bootselect Jumper, J5 Conn_Coaxial, J8 USB_C_Receptacle_USB2.0_16P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

Commit message: As Ordered Aug 4 2025
Routing:
- net 2.8V: track 51.3 -> 26.9 mm
- removed copper zone on In2.Cu, net +3V3
- removed copper zone on In1.Cu, net Dir_Chrg_In
- removed copper zone on In1.Cu, net GND
Other:
- copper layers 4 -> 2
Changed lines of the file:
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@@
 	(layers
 		(0 "F.Cu" signal)
-		(4 "In1.Cu" signal)
-		(6 "In2.Cu" signal)
 		(2 "B.Cu" signal)
 		(9 "F.Adhes" user "F.Adhesive")
@@
 			)
 			(layer "dielectric 1"
-				(type "prepreg")
-				(thickness 0.2104)
-				(material "FR4")
-				(epsilon_r 4.5)
-				(loss_tangent 0.02)
-			)
-			(layer "In1.Cu"
-				(type "copper")
-				(thickness 0.0152)
-			)
-			(layer "dielectric 2"
 				(type "core")
-				(thickness 1.065)
-				(material "FR4")
-				(epsilon_r 4.5)
-				(loss_tangent 0.02)
-			)
-			(layer "In2.Cu"
-				(type "copper")
-				(thickness 0.0152)
-			)
-			(layer "dielectric 3"
-				(type "prepreg")
-				(thickness 0.2104)
+				(thickness 1.5162)
 				(material "FR4")
 				(epsilon_r 4.5)
@@
 	)
 	(segment
-		(start 125.958147 126.607053)
-		(end 125.9458 126.6194)
-		(width 0.1524)
-		(layer "In1.Cu")
-		(net 7)
-	)
-	(segment
-		(start 124.0458 136.8194)
-		(end 123.4188 137.4464)
-		(width 0.254)
-		(layer "In1.Cu")
-		(net 7)
-	)
-	(segment
-		(start 129.8208 126.607053)
-		(end 125.958147 126.607053)
-		(width 0.1524)
-		(layer "In1.Cu")
-		(net 7)
-	)
-	(segment
-		(start 133.2458 124.2194)
-		(end 127.3458 124.2194)
-		(width 0.25)
-		(layer "In1.Cu")
-		(net 7)
-	)
-	(segment
-		(start 127.3458 124.2194)
-		(end 125.7458 122.6194)
-		(width 0.25)
-		(layer "In1.Cu")
-		(net 7)
-	)
-	(segment
-		(start 123.4188 137.4464)
-		(end 118.821594 137.4464)
-		(width 0.254)
-		(layer "In1.Cu")
-		(net 7)
-	)
-	(segment
-		(start 131.1458 124.2194)
-		(end 129.8208 125.5444)
-		(width 0.25)
-		(layer "In1.Cu")
-		(net 7)
-	)
-	(segment
-		(start 129.8208 125.5444)
-		(end 129.8208 126.607053)
-		(width 0.25)
-		(layer "In1.Cu")
-		(net 7)
-	)
-	(segment
-		(start 118.821594 137.4464)
-		(end 118.10673 136.731536)
-		(width 0.254)
-		(layer "In1.Cu")
-		(net 7)
-	)
-	(segment
-		(start 133.2458 124.2194)
-		(end 131.1458 124.2194)
-		(width 0.25)
-		(layer "In1.Cu")
-		(net 7)
-	)
-	(segment
-		(start 133.8458 123.6194)
-		(end 133.2458 124.2194)
-		(width 0.25)
-		(layer "In1.Cu")
-		(net 7)
-	)
-	(segment
 		(start 170.155799 105.1194)
 		(end 171.458299 105.1194)
@@
 		(net 0)
 		(net_name "")
-		(layers "F.Cu" "B.Cu" "In2.Cu")
+		(layers "F.Cu" "B.Cu")
 		(hatch edge 0.5)
 		(connect_pads
@@
 			)
 		)
-	)
-	(zone
-		(net 1)
-		(net_name "GND")
-		(layer "In1.Cu")
-		(name "GND")
-		(hatch edge 0.508)
-		(connect_pads
-			(clearance 0.508)
-		)
-		(min_thickness 0.254)
-		(filled_areas_thickness no)
-		(fill yes
-			(thermal_gap 0.508)
-			(thermal_bridge_width 0.508)
-		)
-		(polygon
-			(pts
-				(xy 216.5858 162.8394) (xy 114.9858 162.8394) (xy 114.9858 61.2394) (xy 216.5858 61.2394)
-			)
-		)
-	)
-	(zone
-		(net 0)
-		(net_name "")
-		(layer "In1.Cu")
-		(hatch edge 0.5)
-		(connect_pads
-			(clearance 0)
-		)
-		(min_thickness 0.25)
-		(filled_areas_thickness no)
-		(keepout
-			(tracks allowed)
-			(vias allowed)
-			(pads allowed)
-			(copperpour not_allowed)
-			(footprints allowed)
-		)
-		(placement
-			(enabled no)
-			(sheetname "")
-		)
-		(fill
-			(thermal_gap 0.5)
-			(thermal_bridge_width 0.5)
-		)
-		(polygon
-			(pts
-				(xy 132.8858 126.8694) (xy 163.4158 126.8694) (xy 163.4158 137.1794) (xy 167.6658 137.1794) (xy 167.6658 126.8694)
-				(xy 197.9158 126.8694) (xy 197.9158 145.5394) (xy 132.8858 145.5394)
-			)
-		)
-	)
-	(zone
-		(net 5)
-		(net_name "Dir_Chrg_In")
-		(layer "In1.Cu")
-		(name "3.3V")
-		(hatch edge 0.508)
-		(priority 1)
-		(connect_pads
-			(clearance 0.508)
-		)
-		(min_thickness 0.254)
-		(filled_areas_thickness no)
-		(fill yes
-			(thermal_gap 0.508)
-			(thermal_bridge_width 0.508)
-		)
-		(polygon
-			(pts
-				(xy 189.5458 107.0194) (xy 114.9858 106.9594) (xy 114.9858 61.2394) (xy 189.5458 61.2194)
-			)
-		)
-	)
-	(zone
-		(net 1)
-		(net_name "GND")
-		(layer "In1.Cu")
-		(hatch edge 0.5)
-		(connect_pads
-			(clearance 0)
-		)
-		(min_thickness 0.25)
-		(filled_areas_thickness no)
-		(fill yes
-			(thermal_gap 0.5)
-			(thermal_bridge_width 0.5)
-		)
-		(polygon
-			(pts
-				(xy 163.4158 126.8694) (xy 163.4158 137.1794) (xy 167.6658 137.1794) (xy 167.6658 126.8694)
-			)
-		)
-	)
-	(zone
-		(net 2)
-		(net_name "+3V3")
-		(layer "In2.Cu")
-		(name "GND2")
-		(hatch edge 0.508)
-		(connect_pads
-			(clearance 0.508)
-		)
-		(min_thickness 0.254)
-		(filled_areas_thickness no)
-		(fill yes
-			(thermal_gap 0.508)
-			(thermal_bridge_width 0.508)
-		)
-		(polygon
-			(pts
-				(xy 216.5858 162.8394) (xy 114.9858 162.8394) (xy 114.9858 61.2394) (xy 216.5858 61.2394)
-			)
-		)
